Commit message: added neo planner and other planner configs

File: src/husky_description/urdf/husky.urdf.xacro (robot description, xacro)
@@ -39,5 +39,5 @@
       <odometry_topic>odom</odometry_topic>
       <odometry_frame>odom</odometry_frame>
-      <odometry_rate>20.0</odometry_rate>
+      <odometry_rate>100.0</odometry_rate>
       <robot_base_frame>base_link</robot_base_frame>
       <publish_odom>true</publish_odom>

File: src/husky_description/urdf/husky_macro.urdf.xacro (robot description, xacro)
@@ -64,5 +64,5 @@
     <link name="${prefix}inertial_link">
       <inertial>
-        <mass value="46.034" />
+        <mass value="10.034" />
         <origin xyz="-0.00065 -0.085 0.062" />
         <inertia ixx="0.6022" ixy="-0.02364" ixz="-0.1197" iyy="1.7386" iyz="-0.001544" izz="2.0296" />
@@ -116,5 +116,5 @@
       </xacro:sensor_arch>
     </xacro:if>
-    <xacro:arg name="gpu" default="false"/>
+    <xacro:arg name="gpu" default="true"/>
     <xacro:property name="gpu" value="$(arg gpu)" />
     <xacro:arg name="organize_cloud" default="false"/>

File: src/husky_description/urdf/wheel.urdf.xacro (robot description, xacro)
@@ -22,9 +22,11 @@
     </link>
     <gazebo reference="${wheel_prefix}_wheel">
-      <mu1 value="1.0"/>
+      <!-- <mu1 value="0.5"/>
       <mu2 value="0.5"/>
       <kp value="10000000.0" />
       <kd value="1.0" />
-      <fdir1 value="1 0 0"/>
+      <fdir1 value="1 0 0"/> -->
+      <mu1>0.0001</mu1>
+      <mu2>0.0001</mu2>
     </gazebo>
     <joint name="${wheel_prefix}_wheel_joint" type="fixed">
@@ -32,4 +34,5 @@
       <child link="${wheel_prefix}_wheel"/>
       <xacro:insert_block name="joint_pose"/>
+      <limit effort="1000.0" lower="-1e+16" upper="1e+16" velocity="15"/>
       <axis xyz="0 1 0" rpy="0 0 0" />
     </joint>
